File: noraneko42c/v1.0/pcb/noraneko42c.kicad_pcb (KiCad board)
At the start: 2 copper layers, 269.7 x 112.2 mm, 145 parts, among them SW1 SW_Push, SW10 SW_Push, SW11 SW_Push, SW12 SW_Push, SW13 SW_Push, SW14 SW_Push, SW15 SW_Push, SW16 SW_Push, SW17 SW_Push, SW18 SW_Push, SW19 SW_Push, SW2 SW_Push, SW20 SW_Push, SW21 SW_Push, SW22 SW_Push, SW23 SW_Push, SW24 SW_Push, SW25 SW_Push, SW26 SW_Push, SW27 SW_Push, SW28 SW_Push, SW29 SW_Push, SW3 SW_Push, SW30 SW_Push, SW31 SW_Push, SW32 SW_Push, SW33 SW_Push, SW34 SW_Push, SW35 SW_Push, SW36 SW_Push, SW37 SW_Push, SW38 SW_Push, SW39 SW_Push, SW4 SW_Push, SW40 SW_Push, SW41 SW_Push, SW42 SW_Push, SW5 SW_Push, SW6 SW_Push, SW7 SW_Push, SW8 SW_Push, SW9 SW_Push, U1 ProMicro

Commit message: noraneko42cをRP2040対応に改造し、Fusion用データを追加
- noraneko42c v1.0 の回路図・基板を改造（PR2040_74th / kbd_SW_PCBA フットプリントを使用）
- 基板の3Dモデル（noraneko42c.step）を追加
- Fusion連携用のKiCadプロジェクト（fusion/noraneko_fusion）を追加

Co-Authored-By: Claude Opus 5.5 <noreply@anthropic.com>
Parts:
- removed LED43, LED44, LED45, LED46, LED47, LED48, LED49, LED50, LED51, LED52, LED53, LED54, LED55, LED56, LED57, LED58, LED59: SK6812MINI-E, Noraneko:SK6812MINI-E
- removed U1: ProMicro, Noraneko:Pro_Micro
- added C1: 100n, Capacitor_SMD:C_0402_1005Metric, B.Cu at (210.9, 143.3)
- added C10: 100n, Capacitor_SMD:C_0402_1005Metric, B.Cu at (215.3, 138.1)
- added C11: 100n, Capacitor_SMD:C_0402_1005Metric, B.Cu at (203.0, 146.4)
- added C12: 20p, Capacitor_SMD:C_0402_1005Metric, B.Cu at (210.2, 159.6)
- added C13: 20p, Capacitor_SMD:C_0402_1005Metric, B.Cu at (207.9, 159.6)
- added C14: 100n, Capacitor_SMD:C_0402_1005Metric, B.Cu at (209.1, 156.4)
- added C15: 10u, Capacitor_SMD:C_0402_1005Metric, B.Cu at (200.2, 135.2)
- added C16: 10u, Capacitor_SMD:C_0402_1005Metric, B.Cu at (200.3, 142.4)
- added C2: 100n, Capacitor_SMD:C_0402_1005Metric, B.Cu at (207.7, 156.4)
- added C3: 1u, Capacitor_SMD:C_0402_1005Metric, B.Cu at (206.2, 144.1)
- added C4: 100n, Capacitor_SMD:C_0402_1005Metric, B.Cu at (209.7, 143.3)
- added C5: 1u, Capacitor_SMD:C_0402_1005Metric, B.Cu at (205.1, 144.1)
- added C6: 100n, Capacitor_SMD:C_0402_1005Metric, B.Cu at (202.9, 151.4)
- added C7: 100n, Capacitor_SMD:C_0402_1005Metric, B.Cu at (215.2, 151.4)
- added C8: 100n, Capacitor_SMD:C_0402_1005Metric, B.Cu at (215.3, 147.4)
- added C9: 100n, Capacitor_SMD:C_0402_1005Metric, B.Cu at (203.0, 145.2)
- added D44: RED, LED_SMD:LED_0402_1005Metric, B.Cu at (197.9, 143.9)
- added J1: 217179-0001, PR2040_74th:Connector_USB-C-Receptacle_SMT_12-Pin_MidMount_Simple, B.Cu at (209.2, 98.7)
- added Q1: BSS138, Package_TO_SOT_SMD:SOT-23, B.Cu at (196.4, 148.4)
- added R10: 1k, Resistor_SMD:R_0402_1005Metric, B.Cu at (221.5, 137.8)
- added R11: 5.1k, Resistor_SMD:R_0402_1005Metric, B.Cu at (200.3, 143.9)
- added R12: 10k, Resistor_SMD:R_0402_1005Metric, B.Cu at (196.4, 151.4)
- added R13: 10k, Resistor_SMD:R_0402_1005Metric, B.Cu at (197.2, 135.2)
- added R4: 5.1k, Resistor_SMD:R_0402_1005Metric, B.Cu at (211.0, 109.9)
- added R5: 27.4, Resistor_SMD:R_0402_1005Metric, B.Cu at (207.4, 144.1)
- added R6: 27.4, Resistor_SMD:R_0402_1005Metric, B.Cu at (208.6, 144.1)
- added R7: 5.1k, Resistor_SMD:R_0402_1005Metric, B.Cu at (207.7, 110.0)
- added R8: 1k, Resistor_SMD:R_0402_1005Metric, B.Cu at (210.4, 156.4)
- added R9: 10k, Resistor_SMD:R_0402_1005Metric, B.Cu at (220.2, 137.8)
- added SW43: SW_Push, Button_Switch_SMD:SW_Push_1P1T_NO_Vertical_Wuerth_434133025816, B.Cu at (217.6, 133.5)
- added U2: RP2040, Package_DFN_QFN:QFN-56-1EP_7x7mm_P0.4mm_EP3.2x3.2mm, B.Cu at (209.2, 150.4)
- added U3: W25Q32JVS, Package_SON:WSON-8-1EP_6x5mm_P1.27mm_EP3.4x4.3mm, B.Cu at (217.5, 141.9)
- added U4: CH213K, PR2040_74th:Package_SOT-23, B.Cu at (201.6, 131.6)
- added U5: AMS1117-3.3, PR2040_74th:Package_SOT-89-3, B.Cu at (200.2, 139.2)
- added Y1: 12M, PR2040_74th:Crystal_SMD_3225-4Pin_3.2x2.5mm_HandSoldering, B.Cu at (209.3, 163.2)
- RESET1: footprint Connector_PinHeader_2.54mm:PinHeader_1x02_P2.54mm_Vertical -> Button_Switch_SMD:SW_Push_1P1T_NO_Vertical_Wuerth_434133025816; moved to B.Cu
- SW1, SW10, SW11, SW12, SW13, SW14, SW15, SW16, SW17, SW18, SW19, SW2, SW20, SW21, SW22, SW23, SW24, SW25, SW26, SW27, SW28, SW29, SW3, SW30, SW31, SW32, SW33, SW34, SW35, SW36, SW37, SW38, SW39, SW4, SW40, SW41, SW42, SW5, SW6, SW7, SW8, SW9: footprint Noraneko:MX_Socket -> kbd_SW_PCBA:Choc_v2_Hotswap_1u; moved to B.Cu
- moved RESET1 29.1 mm to (203.9, 161.2), turned to 90 degrees
- moved D40 9.70 mm to (231.9, 165.0)
- moved D41 9.58 mm to (256.6, 156.8)
- moved D33 9.53 mm to (276.0, 118.6)
- moved D20 9.52 mm to (255.1, 109.7)
- moved D32 9.51 mm to (258.4, 128.5)
- moved D36 9.51 mm to (335.4, 126.5)
- moved D11 9.50 mm to (308.9, 85.7)
- moved D19 9.50 mm to (237.4, 119.6)
- moved D12 9.50 mm to (328.8, 89.0)
- moved D7 9.50 mm to (234.1, 100.8)
- moved D21 9.50 mm to (272.7, 99.8)
- moved D34 9.50 mm to (295.9, 121.9)
- moved D9 9.49 mm to (269.3, 81.2)
- moved D22 9.49 mm to (292.6, 103.1)
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Connections:
- net VCC renamed +5V
- LED1 pad 4: LED -> LED_High_V
- LED42 pad 2: Net-(LED42-Pad2) -> unconnected-(LED42-DOUT-Pad2)
Routing:
- net +5V: track 0.00 -> 1140.2 mm, vias 0 -> 10
- net ROW0: track 0.00 -> 331.0 mm, vias 0 -> 6
- net ROW1: track 0.00 -> 325.1 mm, vias 0 -> 6
- net ROW2: track 0.00 -> 305.2 mm, vias 0 -> 2
- net Net-(LED24-DOUT): track 0.00 -> 278.9 mm, vias 0 -> 2
- net Net-(LED12-DOUT): track 0.00 -> 274.3 mm, vias 0 -> 2
- net Net-(LED36-DOUT): track 0.00 -> 240.1 mm, vias 0 -> 4
- net COL5: track 0.00 -> 196.4 mm, vias 0 -> 8
- net COL4: track 0.00 -> 193.2 mm, vias 0 -> 12
- net COL3: track 0.00 -> 192.3 mm, vias 0 -> 12
- net COL11: track 0.00 -> 186.3 mm, vias 0 -> 2
- net COL0: track 0.00 -> 185.5 mm, vias 0 -> 17
- net ROW3: track 0.00 -> 181.5 mm, vias 0 -> 2
- net COL10: track 0.00 -> 176.5 mm, vias 0 -> 6
- net COL2: track 0.00 -> 169.3 mm, vias 0 -> 12
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- added copper zone on B.Cu, net +1V1
- added copper zone on B.Cu, net +3V3
- removed copper zone on B.Cu, net GND
Other:
- outline, holes or cut-outs redrawn
