File: noraneko42c/v1.0/pcb/noraneko42c.kicad_sch (KiCad schematic)
At the start: 145 parts

Commit message: noraneko42cをRP2040対応に改造し、Fusion用データを追加
- noraneko42c v1.0 の回路図・基板を改造（PR2040_74th / kbd_SW_PCBA フットプリントを使用）
- 基板の3Dモデル（noraneko42c.step）を追加
- Fusion連携用のKiCadプロジェクト（fusion/noraneko_fusion）を追加

Co-Authored-By: Claude Opus 5.5 <noreply@anthropic.com>
Parts:
- removed LED43, LED44, LED45, LED46, LED47, LED48, LED49, LED50, LED51, LED52, LED53, LED54, LED55, LED56, LED57, LED58, LED59: (no value), symbol Noraneko:SK6812MINI-E
- removed U1: (no value), symbol Noraneko:ProMicro
- added C1, C10, C11, C14, C2, C4, C6, C7, C8, C9: 100n, Capacitor_SMD:C_0402_1005Metric, symbol Device:C
- added C12, C13: 20p, Capacitor_SMD:C_0402_1005Metric, symbol Device:C
- added C15, C16: 10u, Capacitor_SMD:C_0402_1005Metric, symbol Device:C
- added C3, C5: 1u, Capacitor_SMD:C_0402_1005Metric, symbol Device:C
- added D44: RED, LED_SMD:LED_0402_1005Metric, symbol Device:LED
- added J1: 217179-0001, PR2040_74th:Connector_USB-C-Receptacle_SMT_12-Pin_MidMount_Simple, symbol 74th_Interface:USB_TypeC-2.0_Receptacle
- added Q1: BSS138, Package_TO_SOT_SMD:SOT-23, symbol Transistor_FET:BSS138
- added R10, R8: 1k, Resistor_SMD:R_0402_1005Metric, symbol Device:R
- added R11, R4, R7: 5.1k, Resistor_SMD:R_0402_1005Metric, symbol Device:R
- added R12, R13, R9: 10k, Resistor_SMD:R_0402_1005Metric, symbol Device:R
- added R5, R6: 27.4, Resistor_SMD:R_0402_1005Metric, symbol Device:R
- added SW43: SW_Push, Button_Switch_SMD:SW_Push_1P1T_NO_Vertical_Wuerth_434133025816, symbol Switch:SW_Push
- added U2: RP2040, Package_DFN_QFN:QFN-56-1EP_7x7mm_P0.4mm_EP3.2x3.2mm, symbol 74th_MCU:RP2040
- added U3: W25Q32JVS, Package_SON:WSON-8-1EP_6x5mm_P1.27mm_EP3.4x4.3mm, symbol 74th_ApplicationIC:W25Q32JVSS-FLASH
- added U4: CH213K, PR2040_74th:Package_SOT-23, symbol 74th_Passive:CH213K_Ideal-Diode-for-USB-Power
- added U5: AMS1117-3.3, PR2040_74th:Package_SOT-89-3, symbol Regulator_Linear:AZ1117-3.3
- added Y1: 12M, PR2040_74th:Crystal_SMD_3225-4Pin_3.2x2.5mm_HandSoldering, symbol 74th_PassiveCommon:Crystal_GND24
- D1, D10, D11, D12, D13, D14, D15, D16, D17, D18, D19, D2, D20, D21, D22, D23, D24, D25, D26, D27, D28, D29, D3, D30, D31, D32, D33, D34, D35, D36, D37, D38, D39, D4, D40, D41, D42, D5, D6, D7, D8, D9: value (none) -> D; footprint (none) -> Noraneko:1N4148W
- LED1, LED10, LED11, LED12, LED13, LED14, LED15, LED16, LED17, LED18, LED19, LED2, LED20, LED21, LED22, LED23, LED24, LED25, LED26, LED27, LED28, LED29, LED3, LED30, LED31, LED32, LED33, LED34, LED35, LED36, LED37, LED38, LED39, LED4, LED40, LED41, LED42, LED5, LED6, LED7, LED8, LED9: value (none) -> SK6812MINI-E; footprint (none) -> Noraneko:SK6812MINI-E
- RESET1: value (none) -> SW_Push; footprint (none) -> Button_Switch_SMD:SW_Push_1P1T_NO_Vertical_Wuerth_434133025816
- SW1, SW10, SW11, SW12, SW13, SW14, SW15, SW16, SW17, SW18, SW19, SW2, SW20, SW21, SW22, SW23, SW24, SW25, SW26, SW27, SW28, SW29, SW3, SW30, SW31, SW32, SW33, SW34, SW35, SW36, SW37, SW38, SW39, SW4, SW40, SW41, SW42, SW5, SW6, SW7, SW8, SW9: value (none) -> SW_Push; footprint (none) -> kbd_SW_PCBA:Choc_v2_Hotswap_1u
Connections:
- net COL0: now also U2.41 (GPIO29_ADC3)
- net COL1: now also U2.40 (GPIO28_ADC2)
- net COL10: now also U2.12 (GPIO9)
- net COL11: now also U2.13 (GPIO10)
- net COL2: now also U2.39 (GPIO27_ADC1)
- net COL3: now also U2.38 (GPIO26_ADC0)
- net COL4: now also U2.37 (GPIO25)
- net COL5: now also U2.36 (GPIO24)
- net COL6: now also U2.6 (GPIO4)
- net COL7: now also U2.7 (GPIO5)
- net COL8: now also U2.8 (GPIO6)
- net COL9: now also U2.11 (GPIO8)
- net GND: now also C1.2, C10.2, C11.2, C12.1, C13.1, C14.2, C15.2, C16.2, C2.2, C3.2, C4.2, C5.2, C6.2, C7.2, C8.2, C9.2, D44.1 (K), J1.4 (GND), R4.2, R7.2, SW43.1, U2.19 (TESTEN), U2.57 (GND), U3.4 (GND), U4.1 (GND), U5.1 (GND), Y1.2, Y1.4
- net ROW0: now also U2.2 (GPIO0)
- net ROW1: now also U2.3 (GPIO1)
- net ROW2: now also U2.4 (GPIO2)
- net ROW3: now also U2.5 (GPIO3)
- net reset: now also U2.26 (RUN)
- net LED renamed LED_High_V
- net LED_High_V: now also Q1.3 (D), R13.1
- net VCC renamed +5V
- net +5V: now also C15.1, R13.2, U4.2 (VO-), U5.3 (VI)
- new net: C13.2, R8.2, Y1.3
- new net: J1.5 (CC1), R7.1
- new net: D44.2 (A), R11.1
- new net: J1.6 (CC2), R4.1
- new net +1V1: C1.1, C2.1, C3.1, U2.23 (DVDD), U2.45 (VREG_VOUT), U2.50 (DVDD)
- new net +3V3: C10.1, C11.1, C14.1, C16.1, C4.1, C5.1, C6.1, C7.1, C8.1, C9.1, Q1.1 (G), R11.2, R12.2, R9.2, U2.1 (IOVDD), U2.10 (IOVDD), U2.22 (IOVDD), U2.33 (IOVDD), U2.42 (IOVDD), U2.43 (ADC_AVDD), U2.44 (VREG_IN), U2.48 (USB_VDD), U2.49 (IOVDD), U3.8 (VCC), U5.2 (VO)
- new net BOOTSEL: R10.1, SW43.2
- new net LED_Low_V: Q1.2 (S), R12.1, U2.27 (GPIO16)
- new net QSPI_CLK: U2.52 (QSPI_SCLK), U3.6 (CLK)
- new net QSPI_SD0: U2.53 (QSPI_SD0), U3.5 (DI(IO0))
- new net QSPI_SD1: U2.55 (QSPI_SD1), U3.2 (DO(IO1))
- new net QSPI_SD2: U2.54 (QSPI_SD2), U3.3 (IO2)
- new net QSPI_SD3: U2.51 (QSPI_SD3), U3.7 (IO3)
- new net QSPI_SS: R10.2, R9.1, U2.56 (QSPI_SS), U3.1 (~{CS})
- new net USB+: J1.3 (D+), R6.1
- new net USB-: J1.2 (D-), R5.1
- new net USB_DN: R5.2, U2.46 (USB_DM)
- new net USB_DP: R6.2, U2.47 (USB_DP)
- new net VBUS: J1.1 (VBUS), U4.3 (VI+)
- new net XIN: C12.2, U2.20 (XIN), Y1.1
- new net XOUT: R8.1, U2.21 (XOUT)
- no-connect marks 3 -> 18
Other:
- note added: "Flash"
- note added: "Oscillator"
- note added: "Power"
- note added: "USB & Power"
- note added: "make sure C3(1u) is close to pin 45 of RP2040"
- note added: "make sure C5(1u) is close to pin 44 of RP2040"
- note added: "make sure R5 and R6 are close to RP2040"
- note added: "レベルシフト回路"
- note removed: "Flags"
- moved on the sheet: LED1, LED10, LED2, LED3, LED31, LED32, LED33, LED34, LED35, LED36, LED37, LED38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
